Commit message: A working ur3 simulation. See ur3_temoto.launch. None of Temoto is enabled in the launch file yet.

File: temoto_universal_robot/ur_description/urdf/ur3_robot.urdf.xacro (robot description, xacro)
@@ -14,3 +14,11 @@
     <origin xyz="0.0 0.0 0.0" rpy="0.0 0.0 0.0" />
   </joint>
+  <!-- attach Temoto frame -->
+  <!-- A tool link that will serve as the end effector, instead of tool0. -->
+  <link name="temoto_end_effector" />
+  <joint name="ur3-temoto" type="fixed" >
+    <origin xyz="0 0 0" rpy="1.571 1.571 -1.571"/>
+    <parent link="ee_link" />
+    <child link="temoto_end_effector" />
+  </joint>
 </robot>
