Commit message: Got the standalone UR5 working. Deleting the deprecated ur3/sia5 stuff. Added an rviz_animated_view_controller submodule.

File: temoto_universal_robot/ur_description/urdf/ur5_robot.urdf.xacro (robot description, xacro)
@@ -18,5 +18,5 @@
   <link name="temoto_end_effector" />
   <joint name="ur5-temoto" type="fixed" >
-    <origin xyz="0.0 0.0 0.0" rpy="0 0 0"/>
+    <origin xyz="0.0 0.0 0.0" rpy="1.571 1.571 -1.571"/>
     <parent link="ee_link" />	<!-- end-effector link for UR5 -->
     <child link="temoto_end_effector" />

Commit message: Fixing the 90 degree rotation for ur5_temoto.launch.

File: temoto_universal_robot/ur_description/urdf/ur5_robot.urdf.xacro (robot description, xacro)
@@ -18,5 +18,5 @@
   <link name="temoto_end_effector" />
   <joint name="ur5-temoto" type="fixed" >
-    <origin xyz="0.0 0.0 0.0" rpy="1.571 1.571 -1.571"/>
+    <origin xyz="0.0 0.0 0.0" rpy="0 -1.571 0"/>
     <parent link="ee_link" />	<!-- end-effector link for UR5 -->
     <child link="temoto_end_effector" />

Commit message: Adding the Woodside gripper to the URDF and updating the SRDF with moveit_setup_assistant.

File: temoto_universal_robot/ur_description/urdf/ur5_robot.urdf.xacro (robot description, xacro)
@@ -22,3 +22,26 @@
     <child link="temoto_end_effector" />
   </joint>
+   <!-- attach gripper. Z is up -->
+  <joint name="hand_attach_joint" type="fixed">
+    <parent link= "ee_link" />
+    <child link = "2_finger_85_gripper_link" />
+    <origin xyz="0.09 0 0" rpy="0 0 -1.571" />
+  </joint>
+  <link name="2_finger_85_gripper_link">
+      <visual>
+        <origin xyz="0 0 0" rpy="0 0 0" />
+        <geometry>
+          <mesh filename="package://temoto_support/meshes/2_finger_85_gripper.stl" scale="0.001 0.001 0.001"/>
+        </geometry>
+        <material name="black">
+          <color rgba="0.05 0.05 0.05 1"/>
+        </material>
+      </visual>
+      <collision>
+        <origin xyz="0.0 0.0 0.0" rpy="0.0 0.0 0.0" />
+        <geometry>
+          <mesh filename="package://temoto_support/meshes/2_finger_85_gripper.stl" scale="0.001 0.001 0.001"/>
+        </geometry>
+      </collision>
+  </link>
 </robot>

Commit message: Got motion planning to work with incremental pose cmds.

File: temoto_universal_robot/ur_description/urdf/ur5_robot.urdf.xacro (robot description, xacro)
@@ -32,5 +32,5 @@
         <origin xyz="0 0 0" rpy="0 0 0" />
         <geometry>
-          <mesh filename="package://temoto_support/meshes/2_finger_85_gripper.stl" scale="0.001 0.001 0.001"/>
+          <mesh filename="package://temoto_support/meshes/2_finger_85_gripper_urdf.stl" scale="0.001 0.001 0.001"/>
         </geometry>
         <material name="black">
@@ -41,5 +41,5 @@
         <origin xyz="0.0 0.0 0.0" rpy="0.0 0.0 0.0" />
         <geometry>
-          <mesh filename="package://temoto_support/meshes/2_finger_85_gripper.stl" scale="0.001 0.001 0.001"/>
+          <mesh filename="package://temoto_support/meshes/2_finger_85_gripper_urdf.stl" scale="0.001 0.001 0.001"/>
         </geometry>
       </collision>

Commit message: Switching to RRT* motion planner (supposedly optimal) and adding a wall and floor to collision scene.

File: temoto_universal_robot/ur_description/urdf/ur5_robot.urdf.xacro (robot description, xacro)
@@ -13,4 +13,48 @@
     <child link = "base_link" />
     <origin xyz="0.0 0.0 0.0" rpy="0.0 0.0 0.0" />
+  </joint>
+  <!-- Floor -->
+  <link name="floor">
+    <collision>
+      <origin xyz="0.0 0.0 0.0" rpy="0.0 0.0 0.0" />
+      <geometry>
+        <box size="3 3 0.01"/>
+      </geometry>
+    </collision>
+    <visual>
+      <geometry>
+        <box size="3 3 0.01"/>
+      </geometry>
+      <material name="transparent_blue">
+        <color rgba="0 0 0.8 0.02"/>
+      </material>
+    </visual>
+  </link>
+  <joint name="world_to_floor" type="fixed">
+    <origin xyz="0 0 -0.1" rpy="0 0 0" />
+    <parent link="world"/>
+    <child link = "floor" />
+  </joint>
+  <!-- Back wall -->
+  <link name="back_wall">
+    <collision>
+      <origin xyz="0.0 0.0 0.0" rpy="0.0 0.0 0.0" />
+      <geometry>
+        <box size="0.01 3 3"/>
+      </geometry>
+    </collision>
+    <visual>
+      <geometry>
+        <box size="0.01 3 3"/>
+      </geometry>
+      <material name="transparent_blue">
+        <color rgba="0 0 0.8 0.02"/>
+      </material>
+    </visual>
+  </link>
+  <joint name="world_to_back_wall" type="fixed">
+    <origin xyz="-0.5 0 1.5" rpy="0 0 0" />
+    <parent link="world"/>
+    <child link = "back_wall" />
   </joint>
   <!-- attach Temoto frame -->

Commit message: Adjusting temoto_end_effector frame since the SpaceNav input coordinates changed.

File: temoto_universal_robot/ur_description/urdf/ur5_robot.urdf.xacro (robot description, xacro)
@@ -62,5 +62,5 @@
   <link name="temoto_end_effector" />
   <joint name="ur5-temoto" type="fixed" >
-    <origin xyz="0.0 0.0 0.0" rpy="0 -1.571 0"/>
+    <origin xyz="0.0 0.0 0.0" rpy="0 0 0"/>
     <parent link="ee_link" />	<!-- end-effector link for UR5 -->
     <child link="temoto_end_effector" />

Commit message: Changing the UR5 control point to the gripper fingers.

File: temoto_universal_robot/ur_description/urdf/ur5_robot.urdf.xacro (robot description, xacro)
@@ -62,5 +62,5 @@
   <link name="temoto_end_effector" />
   <joint name="ur5-temoto" type="fixed" >
-    <origin xyz="0.0 0.0 0.0" rpy="0 0 0"/>
+    <origin xyz="0.15 0.0 0.0" rpy="0 0 0"/>
     <parent link="ee_link" />	<!-- end-effector link for UR5 -->
     <child link="temoto_end_effector" />
