Commit message: Simplifying & moving junk out of main().

File: temoto_universal_robot/ur_description/urdf/ur5.urdf.xacro (robot description, xacro)
@@ -80,5 +80,5 @@
       <collision>
         <geometry>
-          <mesh filename="package://ur_description/meshes/ur5/collision/base.stl" />
+          <mesh filename="package://ur_description/meshes/ur5/collision/base.stl" scale="1.01 1.01 1.01"/>
         </geometry>
       </collision>
@@ -111,5 +111,5 @@
       <collision>
         <geometry>
-          <mesh filename="package://ur_description/meshes/ur5/collision/shoulder.stl" />
+          <mesh filename="package://ur_description/meshes/ur5/collision/shoulder.stl" scale="1.01 1.01 1.01" />
         </geometry>
       </collision>
@@ -142,5 +142,5 @@
       <collision>
         <geometry>
-          <mesh filename="package://ur_description/meshes/ur5/collision/upperarm.stl" />
+          <mesh filename="package://ur_description/meshes/ur5/collision/upperarm.stl" scale="1.01 1.01 1.01" />
         </geometry>
       </collision>
@@ -173,5 +173,5 @@
       <collision>
         <geometry>
-          <mesh filename="package://ur_description/meshes/ur5/collision/forearm.stl" />
+          <mesh filename="package://ur_description/meshes/ur5/collision/forearm.stl" scale="1.01 1.01 1.01" />
         </geometry>
       </collision>
@@ -204,5 +204,5 @@
       <collision>
         <geometry>
-          <mesh filename="package://ur_description/meshes/ur5/collision/wrist1.stl" />
+          <mesh filename="package://ur_description/meshes/ur5/collision/wrist1.stl" scale="1.01 1.01 1.01" />
         </geometry>
       </collision>
@@ -235,5 +235,5 @@
       <collision>
         <geometry>
-          <mesh filename="package://ur_description/meshes/ur5/collision/wrist2.stl" />
+          <mesh filename="package://ur_description/meshes/ur5/collision/wrist2.stl" scale="1.01 1.01 1.01" />
         </geometry>
       </collision>
@@ -266,5 +266,5 @@
       <collision>
         <geometry>
-          <mesh filename="package://ur_description/meshes/ur5/collision/wrist3.stl" />
+          <mesh filename="package://ur_description/meshes/ur5/collision/wrist3.stl" scale="1.01 1.01 1.01"/>
         </geometry>
       </collision>

File: temoto_universal_robot/ur_description/urdf/ur5_robot.urdf.xacro (robot description, xacro)
@@ -85,5 +85,5 @@
         <origin xyz="0.0 0.0 0.0" rpy="0.0 0.0 0.0" />
         <geometry>
-          <mesh filename="package://temoto_support/meshes/2_finger_85_gripper_urdf.stl" scale="0.001 0.001 0.001"/>
+          <mesh filename="package://temoto_support/meshes/2_finger_85_gripper_urdf.stl" scale="0.00105 0.00105 0.00105"/>
         </geometry>
       </collision>

Commit message: Scaling up the stl's in the UR5 collision model.

File: temoto_universal_robot/ur_description/urdf/ur5.urdf.xacro (robot description, xacro)
@@ -80,5 +80,5 @@
       <collision>
         <geometry>
-          <mesh filename="package://ur_description/meshes/ur5/collision/base.stl" scale="1.01 1.01 1.01"/>
+          <mesh filename="package://ur_description/meshes/ur5/collision/base.stl" scale="1.05 1.05 1.05"/>
         </geometry>
       </collision>
@@ -111,5 +111,5 @@
       <collision>
         <geometry>
-          <mesh filename="package://ur_description/meshes/ur5/collision/shoulder.stl" scale="1.01 1.01 1.01" />
+          <mesh filename="package://ur_description/meshes/ur5/collision/shoulder.stl" scale="1.05 1.05 1.05" />
         </geometry>
       </collision>
@@ -142,5 +142,5 @@
       <collision>
         <geometry>
-          <mesh filename="package://ur_description/meshes/ur5/collision/upperarm.stl" scale="1.01 1.01 1.01" />
+          <mesh filename="package://ur_description/meshes/ur5/collision/upperarm.stl" scale="1.05 1.05 1.05" />
         </geometry>
       </collision>
@@ -173,5 +173,5 @@
       <collision>
         <geometry>
-          <mesh filename="package://ur_description/meshes/ur5/collision/forearm.stl" scale="1.01 1.01 1.01" />
+          <mesh filename="package://ur_description/meshes/ur5/collision/forearm.stl" scale="1.05 1.05 1.05" />
         </geometry>
       </collision>
@@ -204,5 +204,5 @@
       <collision>
         <geometry>
-          <mesh filename="package://ur_description/meshes/ur5/collision/wrist1.stl" scale="1.01 1.01 1.01" />
+          <mesh filename="package://ur_description/meshes/ur5/collision/wrist1.stl" scale="1.05 1.05 1.05" />
         </geometry>
       </collision>
@@ -235,5 +235,5 @@
       <collision>
         <geometry>
-          <mesh filename="package://ur_description/meshes/ur5/collision/wrist2.stl" scale="1.01 1.01 1.01" />
+          <mesh filename="package://ur_description/meshes/ur5/collision/wrist2.stl" scale="1.05 1.05 1.05" />
         </geometry>
       </collision>
@@ -266,5 +266,5 @@
       <collision>
         <geometry>
-          <mesh filename="package://ur_description/meshes/ur5/collision/wrist3.stl" scale="1.01 1.01 1.01"/>
+          <mesh filename="package://ur_description/meshes/ur5/collision/wrist3.stl" scale="1.05 1.05 1.05"/>
         </geometry>
       </collision>
